Commit message: clean up

File: src/pr2_description/urdf/gripper_v0/gripper.urdf.xacro (robot description, xacro)
@@ -240,5 +240,5 @@
         <origin xyz="0 0 0" rpy="-1.57 -1 0" />
         <geometry>
-          <mesh filename="package://system_launch/models/mesh/new_stick.dae"   scale="0.15 0.15 0.15" />
+          <mesh filename="package://system_launch/models/mesh/new_stick.dae"   scale="0.17 0.17 0.17" />
         </geometry>
         <material name="Red" />
@@ -247,5 +247,5 @@
         <origin xyz="0 0 0" rpy="-1.57 -1 0" />
         <geometry>
-          <mesh filename="package://system_launch/models/mesh/new_stick.dae"   scale="0.15 0.15 0.15" />
+          <mesh filename="package://system_launch/models/mesh/new_stick.dae"   scale="0.17 0.17 0.17" />
         </geometry>
       </collision>

Commit message: add look for xylophone (turn head)

File: src/pr2_description/urdf/gripper_v0/gripper.urdf.xacro (robot description, xacro)
@@ -240,14 +240,16 @@
         <origin xyz="0 0 0" rpy="-1.57 -1 0" />
         <geometry>
-          <mesh filename="package://system_launch/models/mesh/new_stick.dae"   scale="0.17 0.17 0.17" />
+          <mesh filename="package://system_launch/models/mesh/new_stick.dae"   scale="0.18 0.18 0.18" />
         </geometry>
         <material name="Red" />
       </visual>
+<!--
       <collision>
         <origin xyz="0 0 0" rpy="-1.57 -1 0" />
         <geometry>
-          <mesh filename="package://system_launch/models/mesh/new_stick.dae"   scale="0.17 0.17 0.17" />
-        </geometry>
-      </collision>
+          <mesh filename="package://system_launch/models/mesh/new_stick.dae"   scale="0.23 0.23 0.23" />
+        </geometry>
+      </collision>
+-->
     </link>
     <joint name="${side}_gripper_tool_joint" type="fixed">
